File: ISA-Proto_20201212.kicad_pcb (KiCad board)
At the start: 2 copper layers, 254 x 97.8 mm, 49 parts, among them J1 Conn_01x31_Male, J2 Conn_01x31_Male, J3 Bus_ISA_8bit, J4 Conn_01x31_Male, J5 Conn_01x31_Male

Commit message: Short board version submitted to JLCPCB v0.1
Parts:
- removed the REF** at (153.7, 109.2)
- removed the REF** at (153.7, 68.6)
- removed the REF** at (153.7, 83.8)
- removed the REF** at (153.7, 78.7)
- removed the REF** at (153.7, 104.1)
- removed the REF** at (153.7, 119.4)
- removed the REF** at (153.7, 88.9)
- removed the REF** at (24.1, 53.3)
- removed the REF** at (29.2, 53.3)
- removed the REF** at (34.3, 53.3)
- removed the REF** at (39.4, 53.3)
- removed the REF** at (44.5, 53.3)
- removed the REF** at (49.5, 53.3)
- removed the REF** at (153.7, 124.5)
- removed the REF** at (153.7, 134.6)
- removed the REF** at (153.7, 99.1)
- removed the REF** at (153.7, 129.5)
- removed the REF** at (153.7, 94.0)
- removed the REF** at (153.7, 114.3)
- removed the REF** at (153.7, 53.3)
- removed the REF** at (153.7, 58.4)
- removed the REF** at (153.7, 73.7)
- removed the REF** at (153.7, 63.5)
Other:
- board size 254 x 97.8 mm -> 120.5 x 97.8 mm
- board text added: "8-bit ISA Mini"
- board text added: "FRONT"
- board text added: "REAR"
- board text added: "modified by leadedsolder.com 2022"
- board text removed: "JLCJLCJLCJLC"
